Commit message: slightly change

File: src/tracker_description/description/camera1.xacro (robot description, xacro)
@@ -2,5 +2,5 @@
 <robot xmlns:xacro="http://www.ros.org/wiki/xacro">
     <joint name="camera1_joint" type="fixed">
-        <origin xyz="0.7 0.7 1" rpy="0.0 0.785 -2.36"/>
+        <origin xyz="0.7 0.7 2" rpy="0.0 0.785 -2.36"/>
         <parent link="base_link"/>
         <child link="camera1_link"/>

File: src/tracker_description/description/camera2.xacro (robot description, xacro)
@@ -2,5 +2,5 @@
 <robot xmlns:xacro="http://www.ros.org/wiki/xacro">
     <joint name="camera2_joint" type="fixed">
-        <origin xyz="0.7 -0.7 1" rpy="0.0 0.785 2.36"/>
+        <origin xyz="0.7 -0.7 2" rpy="0.0 0.785 2.36"/>
         <parent link="base_link"/>
         <child link="camera2_link"/>

File: src/tracker_description/description/camera3.xacro (robot description, xacro)
@@ -2,5 +2,5 @@
 <robot xmlns:xacro="http://www.ros.org/wiki/xacro">
     <joint name="camera3_joint" type="fixed">
-        <origin xyz="-0.7 -0.7 1" rpy="0.0 0.785 0.785"/>
+        <origin xyz="-0.7 -0.7 2" rpy="0.0 0.785 0.785"/>
         <parent link="base_link"/>
         <child link="camera3_link"/>

File: src/tracker_description/description/camera4.xacro (robot description, xacro)
@@ -2,5 +2,5 @@
 <robot xmlns:xacro="http://www.ros.org/wiki/xacro">
     <joint name="camera4_joint" type="fixed">
-        <origin xyz="-0.7 0.7 1" rpy="0.0 0.785 -0.785"/>
+        <origin xyz="-0.7 0.7 2" rpy="0.0 0.785 -0.785"/>
         <parent link="base_link"/>
         <child link="camera4_link"/>

Commit message: adjust camera pos and recapture the images

File: src/tracker_description/description/camera1.xacro (robot description, xacro)
@@ -2,5 +2,5 @@
 <robot xmlns:xacro="http://www.ros.org/wiki/xacro">
     <joint name="camera1_joint" type="fixed">
-        <origin xyz="0.7 0.7 2" rpy="0.0 0.785 -2.36"/>
+        <origin xyz="0.4 0.4 1" rpy="0.0 0.785 -2.36"/>
         <parent link="base_link"/>
         <child link="camera1_link"/>

File: src/tracker_description/description/camera2.xacro (robot description, xacro)
@@ -2,5 +2,5 @@
 <robot xmlns:xacro="http://www.ros.org/wiki/xacro">
     <joint name="camera2_joint" type="fixed">
-        <origin xyz="0.7 -0.7 2" rpy="0.0 0.785 2.36"/>
+        <origin xyz="0.4 -0.4 1" rpy="0.0 0.785 2.36"/>
         <parent link="base_link"/>
         <child link="camera2_link"/>

File: src/tracker_description/description/camera3.xacro (robot description, xacro)
@@ -2,5 +2,5 @@
 <robot xmlns:xacro="http://www.ros.org/wiki/xacro">
     <joint name="camera3_joint" type="fixed">
-        <origin xyz="-0.7 -0.7 2" rpy="0.0 0.785 0.785"/>
+        <origin xyz="-0.4 -0.4 1" rpy="0.0 0.785 0.785"/>
         <parent link="base_link"/>
         <child link="camera3_link"/>

File: src/tracker_description/description/camera4.xacro (robot description, xacro)
@@ -2,5 +2,5 @@
 <robot xmlns:xacro="http://www.ros.org/wiki/xacro">
     <joint name="camera4_joint" type="fixed">
-        <origin xyz="-0.7 0.7 2" rpy="0.0 0.785 -0.785"/>
+        <origin xyz="-0.4 0.4 1" rpy="0.0 0.785 -0.785"/>
         <parent link="base_link"/>
         <child link="camera4_link"/>
